Commit message: Setup of URDF and controllers

File: bipedal_description/ros2_control/position_joint_control.ros2_control.xacro (robot description, xacro)
@@ -10,7 +10,4 @@
       </state_interface>
       <state_interface name="effort">
-        <param name="initial_value">0.0</param>
-      </state_interface>
-      <state_interface name="temperature">
         <param name="initial_value">0.0</param>
       </state_interface>

File: bipedal_description/urdf/bipedal.urdf (robot description, URDF)
Before this commit: robot bipedal, 10 links, 9 joints
Links:
- removed link link_foot.L
- removed link link_foot.R
- removed link link_hip
- removed link link_hip_hinge.L
- removed link link_hip_hinge.R
- removed link link_leg.L
- removed link link_leg.R
- removed link link_spine
- removed link link_thigh.L
- removed link link_thigh.R
Joints:
- removed joint foot_joint.L
- removed joint foot_joint.R
- removed joint hip_hinge_joint.L
- removed joint hip_hinge_joint.R
- removed joint leg_joint.L
- removed joint leg_joint.R
- removed joint spine_joint
- removed joint thigh_joint.L
- removed joint thigh_joint.R
