Commit message: Added world link/joint
Got warning from [kdl_parser]: The root link link_hip has an inertia
specified in the URDF, but KDL does not support a root link with an
inertia.  As a workaround, you can add an extra dummy link to your URDF.

File: bipedal_description/urdf/bipedal.urdf (robot description, URDF)
Before this commit: robot bipedal, 0 links, 0 joints
Links:
- added link world
Joints:
- added joint world_joint: type fixed, parent world, child link_hip, origin xyz=0 0 0.964145 rpy=0 0 0
