Commit message: Changed "package://" with "$(find bipedal_description)/"
As noted
[here](https://answers.ros.org/question/401649/gazebo-does-not-spawn-mesh/),
"package://" is no longer supported in ROS 2.

File: bipedal_description/urdf/phobos_generated.urdf (robot description, URDF)
Before this commit: robot reachy_legs, 10 links, 9 joints
Links:
- link link_foot.L: geometry collision box size=0.08800 0.20808 0.08191; visual mesh filename=$(find bipedal_description)/meshes/stl/foot.L.stl scale=1.00000 1.00000 1.00000
- link link_foot.R: geometry collision box size=0.08800 0.20808 0.08191; visual mesh filename=$(find bipedal_description)/meshes/stl/foot.R.stl scale=1.00000 1.00000 1.00000
- link link_hip: geometry collision box size=0.41640 0.13400 0.16853; visual mesh filename=$(find bipedal_description)/meshes/stl/hip.stl scale=1.00000 1.00000 1.00000
- link link_hip_hinge.L: geometry collision box size=0.08800 0.08800 0.20000; visual mesh filename=$(find bipedal_description)/meshes/stl/hip_joint.L.stl scale=1.00000 1.00000 1.00000
- link link_hip_hinge.R: geometry collision box size=0.08800 0.08800 0.20000; visual mesh filename=$(find bipedal_description)/meshes/stl/hip_joint.R.stl scale=1.00000 1.00000 1.00000
- link link_leg.L: geometry collision box size=0.08600 0.16459 0.45010; visual mesh filename=$(find bipedal_description)/meshes/stl/leg.L.stl scale=1.00000 1.00000 1.00000
- link link_leg.R: geometry collision box size=0.08600 0.16459 0.45010; visual mesh filename=$(find bipedal_description)/meshes/stl/leg.R.stl scale=1.00000 1.00000 1.00000
- link link_spine: geometry collision box size=0.09000 0.16247 0.17508; visual mesh filename=$(find bipedal_description)/meshes/stl/spine.stl scale=1.00000 1.00000 1.00000
- link link_thigh.L: geometry collision box size=0.13000 0.20794 0.49535; visual mesh filename=$(find bipedal_description)/meshes/stl/thigh.L.stl scale=1.00000 1.00000 1.00000
- link link_thigh.R: geometry collision box size=0.13000 0.20794 0.49535; visual mesh filename=$(find bipedal_description)/meshes/stl/thigh.R.stl scale=1.00000 1.00000 1.00000

Commit message: Added "file://" so that RViz also can find the meshes

File: bipedal_description/urdf/phobos_generated.urdf (robot description, URDF)
Before this commit: robot reachy_legs, 10 links, 9 joints
Links:
- link link_foot.L: geometry collision box size=0.08800 0.20808 0.08191; visual mesh filename=file://$(find bipedal_description)/meshes/stl/foot.L.stl scale=1.00000 1.00000 1.00000
- link link_foot.R: geometry collision box size=0.08800 0.20808 0.08191; visual mesh filename=file://$(find bipedal_description)/meshes/stl/foot.R.stl scale=1.00000 1.00000 1.00000
- link link_hip: geometry collision box size=0.41640 0.13400 0.16853; visual mesh filename=file://$(find bipedal_description)/meshes/stl/hip.stl scale=1.00000 1.00000 1.00000
- link link_hip_hinge.L: geometry collision box size=0.08800 0.08800 0.20000; visual mesh filename=file://$(find bipedal_description)/meshes/stl/hip_joint.L.s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 scale=1.00000 1.00000 1.00000
- link link_hip_hinge.R: geometry collision box size=0.08800 0.08800 0.20000; visual mesh filename=file://$(find bipedal_description)/meshes/stl/hip_joint.R.s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 scale=1.00000 1.00000 1.00000
- link link_leg.L: geometry collision box size=0.08600 0.16459 0.45010; visual mesh filename=file://$(find bipedal_description)/meshes/stl/leg.L.stl scale=1.00000 1.00000 1.00000
- link link_leg.R: geometry collision box size=0.08600 0.16459 0.45010; visual mesh filename=file://$(find bipedal_description)/meshes/stl/leg.R.stl scale=1.00000 1.00000 1.00000
- link link_spine: geometry collision box size=0.09000 0.16247 0.17508; visual mesh filename=file://$(find bipedal_description)/meshes/stl/spine.stl scale=1.00000 1.00000 1.00000
- link link_thigh.L: geometry collision box size=0.13000 0.20794 0.49535; visual mesh filename=file://$(find bipedal_description)/meshes/stl/thigh.L.stl scale=1.00000 1.00000 1.00000
- link link_thigh.R: geometry collision box size=0.13000 0.20794 0.49535; visual mesh filename=file://$(find bipedal_description)/meshes/stl/thigh.R.stl scale=1.00000 1.00000 1.00000
